Commit message: Add vision grasp pipeline: hand-eye calib, OAK detector, one-shot launcher

File: src/xarm_ros2/xarm_description/urdf/gripper/xarm_gripper.urdf.xacro (robot description, xacro)
@@ -1,5 +1,5 @@
 <?xml version="1.0"?>
 <robot xmlns:xacro="http://ros.org/wiki/xacro" name="xarm_gripper">
-  <xacro:macro name="xarm_gripper_urdf" params="prefix:='' attach_to:='' attach_xyz:='0 0 0' attach_rpy:='0 0 0' ">
+  <xacro:macro name="xarm_gripper_urdf" params="prefix:='' attach_to:='' attach_xyz:='0 0 0' attach_rpy:='0 0 0' replace_finger_meshes:=false ">
     <xacro:unless value="${attach_to == ''}">
       <joint name="${prefix}gripper_fix" type="fixed">
@@ -60,13 +60,26 @@
           iyy="1.7225E-05" iyz="4.6433E-06" izz="5.1466E-06" />
       </inertial>
-      <xacro:common_link_visual
-        mesh_filename="gripper/xarm/left_finger"
-        origin_xyz="0 0 0"
-        origin_rpy="0 0 0"
-        material_name="${prefix}Silver" />
-      <xacro:common_link_collision
-        mesh_filename="gripper/xarm/left_finger"
-        origin_xyz="0 0 0"
-        origin_rpy="0 0 0" />
+      <!--
+        The custom jaw replaces this plate physically.  Keep its mesh as an
+        RViz-only mounting-hole reference, but never as collision geometry.
+      -->
+      <xacro:if value="${replace_finger_meshes}">
+        <xacro:common_link_visual
+          mesh_filename="gripper/xarm/left_finger"
+          origin_xyz="0 0 0"
+          origin_rpy="0 0 0"
+          material_name="${prefix}Silver" />
+      </xacro:if>
+      <xacro:unless value="${replace_finger_meshes}">
+        <xacro:common_link_visual
+          mesh_filename="gripper/xarm/left_finger"
+          origin_xyz="0 0 0"
+          origin_rpy="0 0 0"
+          material_name="${prefix}Silver" />
+        <xacro:common_link_collision
+          mesh_filename="gripper/xarm/left_finger"
+          origin_xyz="0 0 0"
+          origin_rpy="0 0 0" />
+      </xacro:unless>
     </link>
     <joint name="${prefix}left_finger_joint" type="revolute">
@@ -138,13 +151,26 @@
           iyy="1.7225E-05" iyz="-4.6435E-06" izz="5.1466E-06" />
       </inertial>
-      <xacro:common_link_visual
-        mesh_filename="gripper/xarm/right_finger"
-        origin_xyz="0 0 0"
-        origin_rpy="0 0 0"
-        material_name="${prefix}Silver" />
-      <xacro:common_link_collision
-        mesh_filename="gripper/xarm/right_finger"
-        origin_xyz="0 0 0"
-        origin_rpy="0 0 0" />
+      <!--
+        The custom jaw replaces this plate physically.  Keep its mesh as an
+        RViz-only mounting-hole reference, but never as collision geometry.
+      -->
+      <xacro:if value="${replace_finger_meshes}">
+        <xacro:common_link_visual
+          mesh_filename="gripper/xarm/right_finger"
+          origin_xyz="0 0 0"
+          origin_rpy="0 0 0"
+          material_name="${prefix}Silver" />
+      </xacro:if>
+      <xacro:unless value="${replace_finger_meshes}">
+        <xacro:common_link_visual
+          mesh_filename="gripper/xarm/right_finger"
+          origin_xyz="0 0 0"
+          origin_rpy="0 0 0"
+          material_name="${prefix}Silver" />
+        <xacro:common_link_collision
+          mesh_filename="gripper/xarm/right_finger"
+          origin_xyz="0 0 0"
+          origin_rpy="0 0 0" />
+      </xacro:unless>
     </link>
     <joint name="${prefix}right_finger_joint" type="revolute">

File: src/xarm_ros2/xarm_description/urdf/gripper/xarm_gripper_macro.xacro (robot description, xacro)
@@ -7,9 +7,9 @@
   <xacro:include filename="$(find xarm_description)/urdf/gripper/xarm_gripper.gazebo.xacro" />
   <xacro:macro name="xarm_gripper_macro" params="prefix:='' attach_to:='' ns:='xarm' attach_xyz:='0 0 0' attach_rpy:='0 0 0'
-    ros2_control_plugin:='uf_robot_hardware/UFRobotFakeSystemHardware' dof:=7 hard_interface:='PositionJointInterface' ">
+    ros2_control_plugin:='uf_robot_hardware/UFRobotFakeSystemHardware' dof:=7 hard_interface:='PositionJointInterface' replace_finger_meshes:=false ">
     <xacro:if value="${is_ros2 and ros2_control_plugin != 'uf_robot_hardware/UFRobotSystemHardware'}">
       <xacro:xarm_gripper_ros2_control prefix="${prefix}" ros2_control_plugin="${ros2_control_plugin}" />
     </xacro:if>
-    <xacro:xarm_gripper_urdf prefix="${prefix}" attach_to="${attach_to}" attach_xyz="${attach_xyz}" attach_rpy="${attach_rpy}" />
+    <xacro:xarm_gripper_urdf prefix="${prefix}" attach_to="${attach_to}" attach_xyz="${attach_xyz}" attach_rpy="${attach_rpy}" replace_finger_meshes="${replace_finger_meshes}" />
     <xacro:xarm_gripper_transmission prefix="${prefix}" hard_interface="${hard_interface}" />
     <xacro:xarm_gripper_gazebo prefix="${prefix}" />

File: src/xarm_ros2/xarm_description/urdf/xarm_device.urdf.xacro (robot description, xacro)
@@ -7,4 +7,9 @@
   <xacro:arg name="velocity_control" default="false"/>
   <xacro:arg name="add_gripper" default="false"/>
+  <xacro:arg name="add_arc_gripper" default="false"/>
+  <xacro:arg name="arc_gripper_left_xyz" default="0.011717 -0.038337 0.058564"/>
+  <xacro:arg name="arc_gripper_left_rpy" default="0 -1.5707963267948966 0"/>
+  <xacro:arg name="arc_gripper_right_xyz" default="0.010000 0.096583 0.058564"/>
+  <xacro:arg name="arc_gripper_right_rpy" default="0 -1.5707963267948966 0"/>
   <xacro:arg name="add_vacuum_gripper" default="false"/>
   <xacro:arg name="add_bio_gripper" default="false"/>
@@ -21,4 +26,9 @@
   <xacro:arg name="use_gazebo_camera" default="false"/>
   <xacro:arg name="add_other_geometry" default="false"/>
+  <xacro:arg name="add_oak_d_sr" default="false"/>
+  <xacro:arg name="add_oak_d_sr_camera_collision" default="false"/>
+  <xacro:arg name="oak_d_sr_camera_xyz" default="0 0 0"/>
+  <xacro:arg name="oak_d_sr_camera_rpy" default="0 0 0"/>
+  <xacro:arg name="oak_d_sr_camera_safety_radius" default="0.065"/>
   <xacro:arg name="geometry_type" default="box"/>
   <xacro:arg name="geometry_mass" default="0.1"/>
@@ -43,5 +53,8 @@
   <xacro:xarm_device prefix="$(arg prefix)" hw_ns="$(arg hw_ns)" limited="$(arg limited)"
     effort_control="$(arg effort_control)" velocity_control="$(arg velocity_control)"
-    add_gripper="$(arg add_gripper)" add_vacuum_gripper="$(arg add_vacuum_gripper)"
+    add_gripper="$(arg add_gripper)" add_arc_gripper="$(arg add_arc_gripper)"
+    arc_gripper_left_xyz="$(arg arc_gripper_left_xyz)" arc_gripper_left_rpy="$(arg arc_gripper_left_rpy)"
+    arc_gripper_right_xyz="$(arg arc_gripper_right_xyz)" arc_gripper_right_rpy="$(arg arc_gripper_right_rpy)"
+    add_vacuum_gripper="$(arg add_vacuum_gripper)"
     add_bio_gripper="$(arg add_bio_gripper)" dof="$(arg dof)"
     ros2_control_plugin="$(arg ros2_control_plugin)" robot_type="$(arg robot_type)"
@@ -50,4 +63,9 @@
     add_d435i_links="$(arg add_d435i_links)"
     add_other_geometry="$(arg add_other_geometry)"
+    add_oak_d_sr="$(arg add_oak_d_sr)"
+    add_oak_d_sr_camera_collision="$(arg add_oak_d_sr_camera_collision)"
+    oak_d_sr_camera_xyz="$(arg oak_d_sr_camera_xyz)"
+    oak_d_sr_camera_rpy="$(arg oak_d_sr_camera_rpy)"
+    oak_d_sr_camera_safety_radius="$(arg oak_d_sr_camera_safety_radius)"
     geometry_type="$(arg geometry_type)" geometry_mass="$(arg geometry_mass)"
     geometry_height="$(arg geometry_height)" geometry_radius="$(arg geometry_radius)"

File: src/xarm_ros2/xarm_description/urdf/xarm_device_macro.xacro (robot description, xacro)
@@ -8,4 +8,9 @@
     velocity_control:=false
     add_gripper:=false
+    add_arc_gripper:=false
+    arc_gripper_left_xyz:='0.011717 -0.038337 0.058564'
+    arc_gripper_left_rpy:='0 -1.5707963267948966 0'
+    arc_gripper_right_xyz:='0.010000 0.096583 0.058564'
+    arc_gripper_right_rpy:='0 -1.5707963267948966 0'
     add_vacuum_gripper:=false
     add_bio_gripper:=false
@@ -23,4 +28,9 @@
     use_gazebo_camera:=false
     add_other_geometry:=false
+    add_oak_d_sr:=false
+    add_oak_d_sr_camera_collision:=false
+    oak_d_sr_camera_xyz:='0 0 0'
+    oak_d_sr_camera_rpy:='0 0 0'
+    oak_d_sr_camera_safety_radius:='0.065'
     geometry_type:='box'
     geometry_mass:='0.1'
@@ -236,6 +246,19 @@
         <xacro:include filename="$(find xarm_description)/urdf/gripper/xarm_gripper_macro.xacro" />
         <xacro:xarm_gripper_macro prefix="${prefix}" attach_to="${prefix}link_eef"
-          ros2_control_plugin="${ros2_control_plugin}" dof="${dof}" hard_interface="${hard_interface}" />
-      </xacro:unless>
+          ros2_control_plugin="${ros2_control_plugin}" dof="${dof}" hard_interface="${hard_interface}"
+          replace_finger_meshes="${add_arc_gripper}" />
+      </xacro:unless>
+    </xacro:if>
+    <!-- The custom arc jaws are rigidly mounted to the two moving factory fingers. -->
+    <xacro:if value="${add_gripper and add_arc_gripper and robot_type != 'lite'}">
+      <xacro:include filename="$(find xarm_description)/urdf/gripper/arc_gripper_jaws.urdf.xacro" />
+      <xacro:arc_gripper_jaws_urdf
+        prefix="${prefix}"
+        left_finger_link="${prefix}left_finger"
+        right_finger_link="${prefix}right_finger"
+        left_xyz="${arc_gripper_left_xyz}"
+        left_rpy="${arc_gripper_left_rpy}"
+        right_xyz="${arc_gripper_right_xyz}"
+        right_rpy="${arc_gripper_right_rpy}" />
     </xacro:if>
     <xacro:if value="${not add_gripper and add_bio_gripper}">
@@ -271,4 +294,15 @@
       />
     </xacro:if>
+    <xacro:if value="${add_oak_d_sr}">
+      <xacro:include filename="$(find xarm_description)/urdf/camera/oak_d_sr_xarm6.urdf.xacro" />
+      <xacro:oak_d_sr_xarm6_urdf
+        prefix="${prefix}"
+        flange_link="${prefix}link_eef"
+        tcp_link="${prefix}link_tcp"
+        add_camera_collision="${add_oak_d_sr_camera_collision}"
+        camera_xyz="${oak_d_sr_camera_xyz}"
+        camera_rpy="${oak_d_sr_camera_rpy}"
+        camera_safety_radius="${oak_d_sr_camera_safety_radius}" />
+    </xacro:if>
     <!-- gazebo_plugin -->
     <xacro:if value="${load_gazebo_plugin}">

File: src/xarm_ros2/xarm_moveit_config/srdf/_xarm6_macro.srdf.xacro (robot description, xacro)
@@ -10,5 +10,6 @@
   <!-- SUBGROUPS: Groups can also be formed by referencing to already defined group names -->
   <xacro:macro name="xarm6_macro_srdf" params="prefix=''
-    add_gripper='false' add_vacuum_gripper='false' add_bio_gripper='false' add_other_geometry='false' ">
+    add_gripper='false' add_arc_gripper='false' add_vacuum_gripper='false' add_bio_gripper='false' add_other_geometry='false'
+    add_oak_d_sr='false' add_oak_d_sr_camera_collision='false' ">
     <group name="${prefix}xarm6">
       <joint name="${prefix}world_joint" />
@@ -65,4 +66,8 @@
         <link name="${prefix}right_outer_knuckle" />
         <link name="${prefix}right_finger" />
+        <xacro:if value="${add_arc_gripper}">
+          <link name="${prefix}arc_gripper_left_jaw_link" />
+          <link name="${prefix}arc_gripper_right_jaw_link" />
+        </xacro:if>
         <link name="${prefix}link_tcp" />
         <joint name="${prefix}drive_joint" />
@@ -82,4 +87,11 @@
       <passive_joint name="${prefix}right_outer_knuckle_joint" />
       <passive_joint name="${prefix}right_finger_joint" />
+      <xacro:if value="${add_arc_gripper}">
+        <passive_joint name="${prefix}arc_gripper_left_jaw_fix" />
+        <passive_joint name="${prefix}arc_gripper_right_jaw_fix" />
+        <disable_collisions link1="${prefix}arc_gripper_left_jaw_link" link2="${prefix}left_finger" reason="Adjacent" />
+        <disable_collisions link1="${prefix}arc_gripper_right_jaw_link" link2="${prefix}right_finger" reason="Adjacent" />
+        <disable_collisions link1="${prefix}arc_gripper_left_jaw_link" link2="${prefix}arc_gripper_right_jaw_link" reason="Never" />
+      </xacro:if>
       <!-- DISABLE COLLISIONS, By default it is assumed that any link of the robot could potentially come into collision with any other link in the robot. This tag disables collision checking between a specified pair of links. -->
       <disable_collisions link1="${prefix}left_finger" link2="${prefix}left_inner_knuckle" reason="Default" />
@@ -189,4 +201,21 @@
       <disable_collisions link1="${prefix}link_eef" link2="${prefix}other_geometry_link" reason="Adjacent" />
     </xacro:if>
+    <xacro:if value="${add_oak_d_sr}">
+      <passive_joint name="${prefix}oak_d_sr_mount_fix" />
+      <disable_collisions link1="${prefix}link6" link2="${prefix}oak_d_sr_mount_link" reason="Adjacent" />
+      <disable_collisions link1="${prefix}link_eef" link2="${prefix}oak_d_sr_mount_link" reason="Adjacent" />
+      <xacro:if value="${add_gripper}">
+        <disable_collisions link1="${prefix}xarm_gripper_base_link" link2="${prefix}oak_d_sr_mount_link" reason="Default" />
+      </xacro:if>
+      <xacro:if value="${add_oak_d_sr_camera_collision}">
+        <passive_joint name="${prefix}oak_d_sr_camera_fix" />
+        <disable_collisions link1="${prefix}link6" link2="${prefix}oak_rgb_camera_optical_frame" reason="Default" />
+        <disable_collisions link1="${prefix}link_eef" link2="${prefix}oak_rgb_camera_optical_frame" reason="Default" />
+        <xacro:if value="${add_gripper}">
+          <disable_collisions link1="${prefix}xarm_gripper_base_link" link2="${prefix}oak_rgb_camera_optical_frame" reason="Default" />
+          <disable_collisions link1="${prefix}link_tcp" link2="${prefix}oak_rgb_camera_optical_frame" reason="Adjacent" />
+        </xacro:if>
+      </xacro:if>
+    </xacro:if>
     <disable_collisions link1="${prefix}link1" link2="${prefix}link2" reason="Adjacent" />
     <disable_collisions link1="${prefix}link1" link2="${prefix}link3" reason="Never" />

File: src/xarm_ros2/xarm_moveit_config/srdf/xarm.srdf.xacro (robot description, xacro)
@@ -6,9 +6,13 @@
   <xacro:arg name="robot_type" default="xarm" />
   <xacro:arg name="add_gripper" default="false"/>
+  <xacro:arg name="add_arc_gripper" default="false"/>
   <xacro:arg name="add_vacuum_gripper" default="false" />
   <xacro:arg name="add_bio_gripper" default="false" />
   <xacro:arg name="add_other_geometry" default="false" />
+  <xacro:arg name="add_oak_d_sr" default="false" />
+  <xacro:arg name="add_oak_d_sr_camera_collision" default="false" />
   <xacro:include filename="$(find xarm_moveit_config)/srdf/xarm_macro.srdf.xacro" />
   <xacro:xarm_macro_srdf prefix="$(arg prefix)" dof="$(arg dof)" robot_type="$(arg robot_type)"
-    add_gripper="$(arg add_gripper)" add_vacuum_gripper="$(arg add_vacuum_gripper)" add_bio_gripper="$(arg add_bio_gripper)" add_other_geometry="$(arg add_other_geometry)" />
+    add_gripper="$(arg add_gripper)" add_arc_gripper="$(arg add_arc_gripper)" add_vacuum_gripper="$(arg add_vacuum_gripper)" add_bio_gripper="$(arg add_bio_gripper)" add_other_geometry="$(arg add_other_geometry)"
+    add_oak_d_sr="$(arg add_oak_d_sr)" add_oak_d_sr_camera_collision="$(arg add_oak_d_sr_camera_collision)" />
 </robot>

File: src/xarm_ros2/xarm_moveit_config/srdf/xarm_macro.srdf.xacro (robot description, xacro)
@@ -2,5 +2,6 @@
 <robot xmlns:xacro="http://wiki.ros.org/xacro" name="xarm_srdf">
   <xacro:macro name="xarm_macro_srdf" params="prefix:='' dof:=7 robot_type:='xarm'
-    add_gripper:='false' add_vacuum_gripper:='false' add_bio_gripper:='false' add_other_geometry:='false' ">
+    add_gripper:='false' add_arc_gripper:='false' add_vacuum_gripper:='false' add_bio_gripper:='false' add_other_geometry:='false'
+    add_oak_d_sr:='false' add_oak_d_sr_camera_collision:='false' ">
     <xacro:if value="${dof == 5}">
       <xacro:include filename="$(find xarm_moveit_config)/srdf/_xarm5_macro.srdf.xacro" />
@@ -12,5 +13,5 @@
         <xacro:include filename="$(find xarm_moveit_config)/srdf/_uf850_macro.srdf.xacro" />
         <xacro:uf850_macro_srdf prefix="${prefix}"
-          add_gripper="${add_gripper}" add_vacuum_gripper="${add_vacuum_gripper}" add_bio_gripper="${add_bio_gripper}" add_other_geometry="${add_other_geometry}"  />
+          add_gripper="${add_gripper}" add_vacuum_gripper="${add_vacuum_gripper}" add_bio_gripper="${add_bio_gripper}" add_other_geometry="${add_other_geometry}" />
       </xacro:if>
       <xacro:if value="${robot_type == 'lite'}">
@@ -22,5 +23,6 @@
         <xacro:include filename="$(find xarm_moveit_config)/srdf/_xarm6_macro.srdf.xacro" />
         <xacro:xarm6_macro_srdf prefix="${prefix}"
-          add_gripper="${add_gripper}" add_vacuum_gripper="${add_vacuum_gripper}" add_bio_gripper="${add_bio_gripper}" add_other_geometry="${add_other_geometry}"  />
+          add_gripper="${add_gripper}" add_arc_gripper="${add_arc_gripper}" add_vacuum_gripper="${add_vacuum_gripper}" add_bio_gripper="${add_bio_gripper}" add_other_geometry="${add_other_geometry}"
+          add_oak_d_sr="${add_oak_d_sr}" add_oak_d_sr_camera_collision="${add_oak_d_sr_camera_collision}" />
       </xacro:unless>
     </xacro:if>
